Commit message: Rebase from 'release/humble/pmb2_description'

File: robots/pmb2.urdf.xacro (robot description, xacro)
@@ -22,4 +22,6 @@
   <!-- false, true-->
   <xacro:arg name="add_on_module" default="no-add-on"/>
+  <!-- no-camera, orbbec-astra, orbbec-astra-pro, asus-xtion -->
+  <xacro:arg name="camera_model" default="no-camera"/>
   <!-- Execution env config -->
   <xacro:arg name="use_sim_time" default="false"/>
@@ -33,10 +35,14 @@
   <xacro:property name="has_microphone" value="$(arg has_microphone)" />
   <xacro:property name="add_on_module" value="$(arg add_on_module)"/>
+  <xacro:property name="camera_model" value="$(arg camera_model)" />
   <!-- HW configuration check -->
   <xacro:if value="${laser_model not in ['no-laser', 'sick-551', 'sick-561', 'sick-571', 'hokuyo']}">
     <xacro:wrong_laser_model/>
   </xacro:if>
-  <xacro:if value="${add_on_module not in ['no-add-on', 'rgbd-sensors']}">
+  <xacro:if value="${add_on_module not in ['no-add-on', 'cobra']}">
     <xacro:wrong_add_on_module/>
+  </xacro:if>
+  <xacro:if value="${camera_model not in ['no-camera', 'structure']}">
+    <xacro:wrong_camera_model/>
   </xacro:if>
   <!-- Execution env configuration -->
@@ -49,5 +55,5 @@
   <xacro:include filename="$(find pmb2_description)/urdf/base/base_sensors.urdf.xacro" />
   <!-- Courier rgbd sensors -->
-  <xacro:if value="${add_on_module == 'rgbd-sensors'}">
+  <xacro:if value="${add_on_module == 'cobra'}">
     <xacro:include filename="$(find pmb2_description)/urdf/cameras_add_on/cameras_add_on.urdf.xacro" />
   </xacro:if>
@@ -63,5 +69,5 @@
   <xacro:base_sensors name="base" laser_model="${laser_model}" has_sonars="${has_sonars}" has_microphone="${has_microphone}"/>
   <!-- RGBD Sensors -->
-  <xacro:if value="${add_on_module == 'rgbd-sensors'}">
+  <xacro:if value="${add_on_module == 'cobra'}">
     <xacro:cameras_add_on name="cameras_add_on" parent="base_link"/>
   </xacro:if>

File: urdf/sensors/courier.urdf.xacro (robot description, xacro)
@@ -19,7 +19,7 @@
   <xacro:property name="base_rgbd_x" value="0.22697"/>
   <xacro:property name="base_rgbd_y" value="0.0"/>
-  <xacro:property name="base_rgbd_z" value="0.52635"/>
+  <xacro:property name="base_rgbd_z" value="0.535"/>
   <xacro:property name="base_rgbd_R" value="-0.171709"/>
-  <xacro:property name="base_rgbd_P" value="57.9362"/>
+  <xacro:property name="base_rgbd_P" value="60"/>
   <xacro:property name="base_rgbd_Y" value="0.0"/>
   <!-- roof RGBD characteristics -->
@@ -28,5 +28,5 @@
   <xacro:property name="roof_rgbd_z" value="0.470428"/>
   <xacro:property name="roof_rgbd_R" value="-0.299256"/>
-  <xacro:property name="roof_rgbd_P" value="10.596"/>
+  <xacro:property name="roof_rgbd_P" value="12"/>
   <xacro:property name="roof_rgbd_Y" value="0.0"/>
   <!-- RGB characteristics -->
@@ -37,25 +37,27 @@
   <xacro:property name="rgb_P" value="15.0"/>
   <xacro:property name="rgb_Y" value="0.0   "/>
-  <!-- RGBD base -->
-  <xacro:structure_sensor name="base_rgbd_camera" parent="base_link">
-    <!-- Pose of sensor frame wrt to base -->
-    <origin xyz="${base_rgbd_x} ${base_rgbd_y} ${base_rgbd_z}" rpy="${base_rgbd_R * deg_to_rad} ${base_rgbd_P * deg_to_rad} ${base_rgbd_Y * deg_to_rad}"/>
-    <!-- Pose of optical frame wrt to sensor -->
-    <origin xyz="0 0 0" rpy="${-90 * deg_to_rad} 0 ${-90 * deg_to_rad}"/>
-  </xacro:structure_sensor>
-  <!-- RGBD roof -->
-  <xacro:structure_sensor name="roof_rgbd_camera" parent="base_link">
-    <!-- Pose of sensor frame wrt to base -->
-    <origin xyz="${roof_rgbd_x} ${roof_rgbd_y} ${roof_rgbd_z}" rpy="${roof_rgbd_R * deg_to_rad} ${roof_rgbd_P * deg_to_rad} ${roof_rgbd_Y * deg_to_rad}"/>
-    <!-- Pose of optical frame wrt to sensor -->
-    <origin xyz="0 0 0" rpy="${-90 * deg_to_rad} 0 ${-90 * deg_to_rad}"/>
-  </xacro:structure_sensor>
-  <!-- RGB -->
-  <xacro:elp_rgb name="rgb_camera" parent="base_link">
-    <!-- Pose of sensor frame wrt to base -->
-    <origin xyz="${rgb_x} ${rgb_y} ${rgb_z}" rpy="${rgb_R * deg_to_rad} ${rgb_P * deg_to_rad} ${rgb_Y * deg_to_rad}"/>
-    <!-- Pose of optical frame wrt to sensor -->
-    <origin xyz="0 0 0" rpy="${-90 * deg_to_rad} 0 ${-90 * deg_to_rad}"/>
-  </xacro:elp_rgb>
+  <xacro:if value="${camera_model == 'structure'}">
+    <!-- RGBD base -->
+    <xacro:structure_sensor name="base_rgbd_camera" parent="base_link">
+      <!-- Pose of sensor frame wrt to base -->
+      <origin xyz="${base_rgbd_x} ${base_rgbd_y} ${base_rgbd_z}" rpy="${base_rgbd_R * deg_to_rad} ${base_rgbd_P * deg_to_rad} ${base_rgbd_Y * deg_to_rad}"/>
+      <!-- Pose of optical frame wrt to sensor -->
+      <origin xyz="0 0 0" rpy="${-90 * deg_to_rad} 0 ${-90 * deg_to_rad}"/>
+    </xacro:structure_sensor>
+    <!-- RGBD roof -->
+    <xacro:structure_sensor name="roof_rgbd_camera" parent="base_link">
+      <!-- Pose of sensor frame wrt to base -->
+      <origin xyz="${roof_rgbd_x} ${roof_rgbd_y} ${roof_rgbd_z}" rpy="${roof_rgbd_R * deg_to_rad} ${roof_rgbd_P * deg_to_rad} ${roof_rgbd_Y * deg_to_rad}"/>
+      <!-- Pose of optical frame wrt to sensor -->
+      <origin xyz="0 0 0" rpy="${-90 * deg_to_rad} 0 ${-90 * deg_to_rad}"/>
+    </xacro:structure_sensor>
+    <!-- RGB -->
+    <xacro:elp_rgb name="rgb_camera" parent="base_link">
+      <!-- Pose of sensor frame wrt to base -->
+      <origin xyz="${rgb_x} ${rgb_y} ${rgb_z}" rpy="${rgb_R * deg_to_rad} ${rgb_P * deg_to_rad} ${rgb_Y * deg_to_rad}"/>
+      <!-- Pose of optical frame wrt to sensor -->
+      <origin xyz="0 0 0" rpy="${-90 * deg_to_rad} 0 ${-90 * deg_to_rad}"/>
+    </xacro:elp_rgb>
+  </xacro:if>
   <!-- RGBD Laser Link -->
   <joint name="rgbd_laser_joint" type="fixed">

File: urdf/sensors/elp_rgb.gazebo.xacro (robot description, xacro)
@@ -16,5 +16,6 @@
     <gazebo reference="${name}_link">
       <!-- RGB -->
-      <sensor type="depth" name="${name}_frame_sensor">
+      <sensor type="camera" name="${name}_frame_sensor">
+        <always_on>true</always_on>
         <update_rate>30.0</update_rate>
         <camera>
@@ -34,17 +35,48 @@
             <stddev>0.007</stddev>
           </noise>
+          <distortion>
+            <k1>0.0</k1>
+            <k2>0.0</k2>
+            <k3>0.0</k3>
+            <p1>0.0</p1>
+            <p2>0.0</p2>
+          </distortion>
         </camera>
         <plugin name="${name}_frame_controller" filename="libgazebo_ros_camera.so">
-          <alwaysOn>true</alwaysOn>
-          <updateRate>0.0</updateRate>
-          <cameraName>${name}</cameraName>
-          <imageTopicName>rgb/image_raw</imageTopicName>
-          <cameraInfoTopicName>rgb/camera_info</cameraInfoTopicName>
-          <frameName>${name}_link</frameName>
-          <distortionK1>0.0</distortionK1>
-          <distortionK2>0.0</distortionK2>
-          <distortionK3>0.0</distortionK3>
-          <distortionT1>0.0</distortionT1>
-          <distortionT2>0.0</distortionT2>
+          <camera_name>${name}</camera_name>
+          <frame_name>${name}_link</frame_name>
+          <ros>
+            <remapping>${name}/image_raw:=${name}/rgb/image_raw</remapping>
+            <remapping>${name}/camera_info:=${name}/rgb/camera_info</remapping>
+            <remapping>${name}/image_raw/compressed:=${name}/rgb/image_raw/compressed</remapping>
+            <remapping>${name}/image_raw/compressedDepth:=${name}/rgb/image_raw/compressedDepth</remapping>
+            <remapping>${name}/image_raw/theora:=${name}/rgb/image_raw/theora</remapping>
+            <qos>
+              <topic name="${name}/rgb/image_raw">
+                <publisher>
+                  <reliability>best_effort</reliability>
+                  <durability>volatile</durability>
+                  <history depth="1">keep_last</history>
+                  <liveliness>automatic</liveliness>
+                </publisher>
+              </topic>
+              <topic name="${name}/rgb/image_raw/compressed">
+                <publisher>
+                  <reliability>best_effort</reliability>
+                  <durability>volatile</durability>
+                  <history depth="1">keep_last</history>
+                  <liveliness>automatic</liveliness>
+                </publisher>
+              </topic>
+              <topic name="${name}/rgb/image_raw/compressedDepth">
+                <publisher>
+                  <reliability>best_effort</reliability>
+                  <durability>volatile</durability>
+                  <history depth="1">keep_last</history>
+                  <liveliness>automatic</liveliness>
+                </publisher>
+              </topic>
+            </qos>
+          </ros>
         </plugin>
       </sensor>

File: urdf/sensors/structure_sensor.gazebo.xacro (robot description, xacro)
@@ -30,55 +30,82 @@
             <far>10.0</far>
           </clip>
+          <distortion>
+            <k1>0.0</k1>
+            <k2>0.0</k2>
+            <k3>0.0</k3>
+            <p1>0.0</p1>
+            <p2>0.0</p2>
+          </distortion>
         </camera>
-        <plugin name="${name}_frame_controller" filename="libgazebo_ros_openni_kinect.so">
-          <alwaysOn>true</alwaysOn>
-          <updateRate>6.0</updateRate>
-          <cameraName>${name}</cameraName>
-          <imageTopicName>ir/image_raw</imageTopicName>
-          <cameraInfoTopicName>ir/camera_info</cameraInfoTopicName>
-          <depthImageTopicName>depth/image_raw</depthImageTopicName>
-          <depthImageCameraInfoTopicName>depth/camera_info</depthImageCameraInfoTopicName>
-          <pointCloudTopicName>depth/points</pointCloudTopicName>
-          <frameName>${name}_optical_frame</frameName>
-          <pointCloudCutoff>0.45</pointCloudCutoff>
-          <rangeMax>10.0</rangeMax>
-          <distortionK1>0.00000001</distortionK1>
-          <distortionK2>0.00000001</distortionK2>
-          <distortionK3>0.00000001</distortionK3>
-          <distortionT1>0.00000001</distortionT1>
-          <distortionT2>0.00000001</distortionT2>
-        </plugin>
-      </sensor>
-      <!-- RGB -->
-      <sensor type="depth" name="${name}_frame_sensor">
-        <always_on>true</always_on>
-        <update_rate>6.0</update_rate>
-        <camera>
-          <horizontal_fov>${58.0 * deg_to_rad}</horizontal_fov>
-          <image>
-            <format>R8G8B8</format>
-            <width>320</width>
-            <height>240</height>
-          </image>
-          <clip>
-            <near>0.45</near>
-            <far>10.0</far>
-          </clip>
-        </camera>
-        <plugin name="${name}_frame_controller" filename="libgazebo_ros_openni_kinect.so">
-          <alwaysOn>true</alwaysOn>
-          <updateRate>6.0</updateRate>
-          <cameraName>${name}</cameraName>
-          <imageTopicName>rgb/image_raw</imageTopicName>
-          <cameraInfoTopicName>rgb/camera_info</cameraInfoTopicName>
-          <pointCloudTopicName>rgb/points</pointCloudTopicName>
-          <frameName>${name}_optical_frame</frameName>
-          <pointCloudCutoff>0.45</pointCloudCutoff>
-          <rangeMax>10.0</rangeMax>
-          <distortionK1>0.00000001</distortionK1>
-          <distortionK2>0.00000001</distortionK2>
-          <distortionK3>0.00000001</distortionK3>
-          <distortionT1>0.00000001</distortionT1>
-          <distortionT2>0.00000001</distortionT2>
+        <plugin name="${name}_ir" filename="libgazebo_ros_camera.so">
+          <camera_name>${name}</camera_name>
+          <frame_name>${name}_optical_frame</frame_name>
+          <max_depth>10.0</max_depth>
+          <ros>
+            <remapping>${name}/image_raw:=${name}/ir/image_raw</remapping>
+            <remapping>${name}/camera_info:=${name}/ir/camera_info</remapping>
+            <remapping>${name}/image_raw/compressed:=${name}/ir/image_raw/compressed</remapping>
+            <remapping>${name}/image_raw/compressedDepth:=${name}/ir/image_raw/compressedDepth</remapping>
+            <remapping>${name}/image_raw/theora:=${name}/ir/image_raw/theora</remapping>
+            <remapping>${name}/points:=${name}/depth/points</remapping>
+            <qos>
+              <topic name="${name}/ir/image_raw">
+                <publisher>
+                  <reliability>best_effort</reliability>
+                  <durability>volatile</durability>
+                  <history depth="1">keep_last</history>
+                  <liveliness>automatic</liveliness>
+                </publisher>
+              </topic>
+              <topic name="${name}/ir/image_raw/compressed">
+                <publisher>
+                  <reliability>best_effort</reliability>
+                  <durability>volatile</durability>
+                  <history depth="1">keep_last</history>
+                  <liveliness>automatic</liveliness>
+                </publisher>
+              </topic>
+              <topic name="${name}/ir/image_raw/compressedDepth">
+                <publisher>
+                  <reliability>best_effort</reliability>
+                  <durability>volatile</durability>
+                  <history depth="1">keep_last</history>
+                  <liveliness>automatic</liveliness>
+                </publisher>
+              </topic>
+              <topic name="${name}/depth/image_raw">
+                <publisher>
+                  <reliability>best_effort</reliability>
+                  <durability>volatile</durability>
+                  <history depth="1">keep_last</history>
+                  <liveliness>automatic</liveliness>
+                </publisher>
+              </topic>
+              <topic name="${name}/depth/image_raw/compressed">
+                <publisher>
+                  <reliability>best_effort</reliability>
+                  <durability>volatile</durability>
+                  <history depth="1">keep_last</history>
+                  <liveliness>automatic</liveliness>
+                </publisher>
+              </topic>
+              <topic name="${name}/depth/image_raw/compressedDepth">
+                <publisher>
+                  <reliability>best_effort</reliability>
+                  <durability>volatile</durability>
+                  <history depth="1">keep_last</history>
+                  <liveliness>automatic</liveliness>
+                </publisher>
+              </topic>
+              <topic name="${name}/depth/points">
+                <publisher>
+                  <reliability>best_effort</reliability>
+                  <durability>volatile</durability>
+                  <history depth="1">keep_last</history>
+                  <liveliness>automatic</liveliness>
+                </publisher>
+              </topic>
+            </qos>
+          </ros>
         </plugin>
       </sensor>
