Commit message: Imported upstream version '5.10.2' of 'upstream'

File: pmb2_description/urdf/base/base.urdf.xacro (robot description, xacro)
@@ -19,5 +19,6 @@
   <xacro:property name="wheel_separation" value="0.4044"/>
   <xacro:property name="wheel_torque" value="6.0"/>
-  <xacro:property name="wheel_velocity" value="1.0"/>
+  <!-- TODO Compute real wheel max velocity -->
+  <xacro:property name="wheel_velocity" value="100.0"/>
   <!-- Caster wheel characteristics -->
   <xacro:property name="caster_radius" value="0.025"/>

File: pmb2_description/urdf/wheels/wheel.ros2_control.xacro (robot description, xacro)
@@ -13,10 +13,8 @@
  -->
 <robot xmlns:xacro="http://ros.org/wiki/xacro">
+  <!-- TODO Compute real wheel max velocity -->
   <xacro:macro name="ros2_control_wheel" params="side">
     <joint name="wheel_${side}_joint">
-      <command_interface name="velocity">
-        <param name="min">-1</param>
-        <param name="max">1</param>
-      </command_interface>
+      <command_interface name="velocity" />
       <state_interface name="position" />
     </joint>

File: pmb2_description/urdf/wheels/wheel.urdf.xacro (robot description, xacro)
@@ -55,5 +55,5 @@
       <origin xyz="0 ${-separation / 2 * reflect} 0.0" rpy="${-90.0 * deg_to_rad} 0 0"/>
       <axis xyz="0 0 1"/>
-      <limit effort="${torque}" velocity="${velocity / radius}"/>
+      <limit effort="${torque}" velocity="${velocity}"/>
       <dynamics damping="1.0" friction="2.0"/>
     </joint>
