Commit message: Imported upstream version '5.9.0' of 'upstream'

File: pmb2_description/robots/pmb2.urdf.xacro (robot description, xacro)
@@ -26,5 +26,4 @@
   <!-- Execution env config -->
   <xacro:arg name="use_sim_time" default="false"/>
-  <xacro:arg name="is_multiple" default="false"/>
   <xacro:arg name="namespace" default=""/>
   <xacro:arg name="is_public_sim" default="false"/>
@@ -48,5 +47,4 @@
   <!-- Execution env configuration -->
   <xacro:property name="use_sim_time" default="$(arg use_sim_time)"/>
-  <xacro:property name="is_multiple" value="$(arg is_multiple)" />
   <xacro:property name="namespace" value="$(arg namespace)" />
   <xacro:property name="is_public_sim" value="$(arg is_public_sim)" />

File: pmb2_description/ros2_control/ros2_control.urdf.xacro (robot description, xacro)
@@ -15,5 +15,4 @@
   <!-- INCLUDES -->
   <xacro:include filename="$(find pmb2_description)/urdf/wheels/wheel.ros2_control.xacro"/>
-  <xacro:include filename="$(find pmb2_description)/urdf/sensors/sensors.ros2_control.xacro"/>
   <!-- MACRO DEFINITION-->
   <xacro:macro name="pmb2_ros2_control">
@@ -22,4 +21,9 @@
       <gazebo>
         <plugin filename="libgazebo_ros2_control.so" name="gazebo_ros2_control">
+          <ros>
+            <namespace>${namespace}</namespace>
+            <remapping>/tf:=tf</remapping>
+            <remapping>/tf_static:=tf_static</remapping>
+          </ros>
           <parameters>$(find pmb2_description)/ros2_control/gazebo_controller_manager_cfg.yaml</parameters>
         </plugin>

File: pmb2_description/urdf/base/base.gazebo.xacro (robot description, xacro)
@@ -33,11 +33,11 @@
     <gazebo>
       <plugin filename="libgazebo_world_odometry.so" name="gazebo_ros_odometry">
+        <ros>
+          <namespace>${namespace}</namespace>
+        </ros>
         <frame_name>world</frame_name>
         <body_name>base_footprint</body_name>
         <topic_name>ground_truth_odom</topic_name>
         <update_rate>100.0</update_rate>
-        <xacro:if value="${is_multiple}">
-          <namespace>/${nsp}</namespace>
-        </xacro:if>
       </plugin>
     </gazebo>

File: pmb2_description/urdf/base/base_sensors.urdf.xacro (robot description, xacro)
@@ -19,11 +19,11 @@
   <!-- INCLUDES -->
   <xacro:include filename="$(find pmb2_description)/urdf/base/base.urdf.xacro"/>
-  <xacro:include filename="$(find pmb2_description)/urdf/sensors/imu.urdf.xacro"/>
-  <xacro:include filename="$(find pmb2_description)/urdf/sensors/hokuyo_urg_04lx_ug01_laser.urdf.xacro"/>
-  <xacro:include filename="$(find pmb2_description)/urdf/sensors/sick_tim551_laser.urdf.xacro"/>
-  <xacro:include filename="$(find pmb2_description)/urdf/sensors/sick_tim561_laser.urdf.xacro"/>
-  <xacro:include filename="$(find pmb2_description)/urdf/sensors/sick_tim571_laser.urdf.xacro"/>
-  <xacro:include filename="$(find pmb2_description)/urdf/sensors/range.urdf.xacro"/>
-  <xacro:include filename="$(find pmb2_description)/urdf/sensors/microphone.urdf.xacro"/>
+  <xacro:include filename="$(find pal_urdf_utils)/urdf/interaction_sensors/imu.urdf.xacro"/>
+  <xacro:include filename="$(find pal_urdf_utils)/urdf/laser/hokuyo_urg_04lx_ug01_laser.urdf.xacro"/>
+  <xacro:include filename="$(find pal_urdf_utils)/urdf/laser/sick_tim551_laser.urdf.xacro"/>
+  <xacro:include filename="$(find pal_urdf_utils)/urdf/laser/sick_tim561_laser.urdf.xacro"/>
+  <xacro:include filename="$(find pal_urdf_utils)/urdf/laser/sick_tim571_laser.urdf.xacro"/>
+  <xacro:include filename="$(find pal_urdf_utils)/urdf/laser/range.urdf.xacro"/>
+  <xacro:include filename="$(find pal_urdf_utils)/urdf/interaction_sensors/microphone.urdf.xacro"/>
   <!-- MACRO DEFINITION -->
   <xacro:macro name="base_sensors" params="name laser_model:=sick-571 has_sonars:=false has_microphone:=false" >

File: pmb2_description/urdf/cameras_add_on/cameras_add_on.urdf.xacro (robot description, xacro)
@@ -13,6 +13,64 @@
 -->
 <robot xmlns:xacro="http://ros.org/wiki/xacro">
-  <!-- INCLUDES -->
-  <xacro:include filename="$(find pmb2_description)/urdf/sensors/courier.urdf.xacro" />
+  <xacro:include filename="$(find pal_urdf_utils)/urdf/camera/structure_sensor.urdf.xacro"/>
+  <xacro:include filename="$(find pal_urdf_utils)/urdf/camera/elp_rgb.urdf.xacro"/>
+  <xacro:include filename="$(find pal_urdf_utils)/urdf/deg_to_rad.urdf.xacro" />
+  <!-- base RGBD characteristics -->
+  <xacro:property name="base_rgbd_x" value="0.22697"/>
+  <xacro:property name="base_rgbd_y" value="0.0"/>
+  <xacro:property name="base_rgbd_z" value="0.535"/>
+  <xacro:property name="base_rgbd_R" value="-0.171709"/>
+  <xacro:property name="base_rgbd_P" value="60"/>
+  <xacro:property name="base_rgbd_Y" value="0.0"/>
+  <!-- roof RGBD characteristics -->
+  <xacro:property name="roof_rgbd_x" value="0.18473"/>
+  <xacro:property name="roof_rgbd_y" value="0.0"/>
+  <xacro:property name="roof_rgbd_z" value="0.470428"/>
+  <xacro:property name="roof_rgbd_R" value="-0.299256"/>
+  <xacro:property name="roof_rgbd_P" value="12"/>
+  <xacro:property name="roof_rgbd_Y" value="0.0"/>
+  <!-- RGB characteristics -->
+  <xacro:property name="rgb_x" value="0.18752"/>
+  <xacro:property name="rgb_y" value="0.0"/>
+  <xacro:property name="rgb_z" value="0.3301"/>
+  <xacro:property name="rgb_R" value="0.0"/>
+  <xacro:property name="rgb_P" value="15.0"/>
+  <xacro:property name="rgb_Y" value="0.0   "/>
+  <xacro:if value="${camera_model == 'structure'}">
+    <!-- RGBD base -->
+    <xacro:structure_sensor name="base_rgbd_camera" parent="base_link">
+      <!-- Pose of sensor frame wrt to base -->
+      <origin xyz="${base_rgbd_x} ${base_rgbd_y} ${base_rgbd_z}" rpy="${base_rgbd_R * deg_to_rad} ${base_rgbd_P * deg_to_rad} ${base_rgbd_Y * deg_to_rad}"/>
+      <!-- Pose of optical frame wrt to sensor -->
+      <origin xyz="0 0 0" rpy="${-90 * deg_to_rad} 0 ${-90 * deg_to_rad}"/>
+    </xacro:structure_sensor>
+    <!-- RGBD roof -->
+    <xacro:structure_sensor name="roof_rgbd_camera" parent="base_link">
+      <!-- Pose of sensor frame wrt to base -->
+      <origin xyz="${roof_rgbd_x} ${roof_rgbd_y} ${roof_rgbd_z}" rpy="${roof_rgbd_R * deg_to_rad} ${roof_rgbd_P * deg_to_rad} ${roof_rgbd_Y * deg_to_rad}"/>
+      <!-- Pose of optical frame wrt to sensor -->
+      <origin xyz="0 0 0" rpy="${-90 * deg_to_rad} 0 ${-90 * deg_to_rad}"/>
+    </xacro:structure_sensor>
+    <!-- RGB -->
+    <xacro:elp_rgb name="rgb_camera" parent="base_link">
+      <!-- Pose of sensor frame wrt to base -->
+      <origin xyz="${rgb_x} ${rgb_y} ${rgb_z}" rpy="${rgb_R * deg_to_rad} ${rgb_P * deg_to_rad} ${rgb_Y * deg_to_rad}"/>
+      <!-- Pose of optical frame wrt to sensor -->
+      <origin xyz="0 0 0" rpy="${-90 * deg_to_rad} 0 ${-90 * deg_to_rad}"/>
+    </xacro:elp_rgb>
+  </xacro:if>
+  <!-- RGBD Laser Link -->
+  <joint name="rgbd_laser_joint" type="fixed">
+    <parent link="base_footprint"/>
+    <child link="rgbd_laser_link"/>
+    <origin xyz="-0.9 0 0" rpy="0 0 0" />
+  </joint>
+  <link name="rgbd_laser_link">
+    <inertial>
+      <origin xyz="0 0 0" rpy="0 0 0"/>
+      <mass value="0.0001" />
+      <inertia ixx="0.0001" ixy="0" ixz="0" iyy="0.0001" iyz="0" izz="0.0001" />
+    </inertial>
+  </link>
   <!-- MACRO DEFINITION-->
   <xacro:macro name="cameras_add_on" params="name parent">

Commit message: Imported upstream version '5.11.2' of 'upstream'

File: pmb2_description/robots/pmb2.urdf.xacro (robot description, xacro)
@@ -28,4 +28,5 @@
   <xacro:arg name="namespace" default=""/>
   <xacro:arg name="is_public_sim" default="false"/>
+  <xacro:arg name="gazebo_version" default="classic"/>
   <!-- PROPERTIES -->
   <!-- HW configuration -->
@@ -49,4 +50,5 @@
   <xacro:property name="namespace" value="$(arg namespace)" />
   <xacro:property name="is_public_sim" value="$(arg is_public_sim)" />
+  <xacro:property name="gazebo_version" value="$(arg gazebo_version)" />
   <!-- INCLUDES -->
   <!-- Base -->

File: pmb2_description/ros2_control/ros2_control.urdf.xacro (robot description, xacro)
@@ -20,12 +20,21 @@
     <xacro:if value="${use_sim_time}">
       <gazebo>
-        <plugin filename="libgazebo_ros2_control.so" name="gazebo_ros2_control">
-          <ros>
-            <namespace>${namespace}</namespace>
-            <remapping>/tf:=tf</remapping>
-            <remapping>/tf_static:=tf_static</remapping>
-          </ros>
-          <parameters>$(find pmb2_description)/ros2_control/gazebo_controller_manager_cfg.yaml</parameters>
-        </plugin>
+        <xacro:if value="${gazebo_version == 'classic'}">
+          <plugin filename="libgazebo_ros2_control.so" name="gazebo_ros2_control">
+            <ros>
+              <namespace>${namespace}</namespace>
+              <remapping>/tf:=tf</remapping>
+              <remapping>/tf_static:=tf_static</remapping>
+            </ros>
+            <parameters>$(find pmb2_description)/ros2_control/gazebo_controller_manager_cfg.yaml</parameters>
+          </plugin>
+        </xacro:if>
+        <xacro:if value="${gazebo_version == 'gazebo'}">
+          <plugin filename="gz_ros2_control-system" name="gz_ros2_control::GazeboSimROS2ControlPlugin">
+            <robot_param>robot_description</robot_param>
+            <robot_param_node>robot_state_publisher</robot_param_node>
+            <parameters>$(find pmb2_description)/ros2_control/gazebo_controller_manager_cfg.yaml</parameters>
+          </plugin>
+        </xacro:if>
       </gazebo>
     </xacro:if>
@@ -36,5 +45,10 @@
         <!-- HW interface gazebo-->
         <hardware>
-          <plugin>gazebo_ros2_control/GazeboSystem</plugin>
+          <xacro:if value="${gazebo_version == 'classic'}">
+            <plugin>gazebo_ros2_control/GazeboSystem</plugin>
+          </xacro:if>
+          <xacro:if value="${gazebo_version == 'gazebo'}">
+            <plugin>gz_ros2_control/GazeboSimSystem</plugin>
+          </xacro:if>
         </hardware>
       </xacro:if>

File: pmb2_description/urdf/base/base.gazebo.xacro (robot description, xacro)
@@ -32,13 +32,15 @@
     <!-- Odometry plugin for ground truth -->
     <gazebo>
-      <plugin filename="libgazebo_world_odometry.so" name="gazebo_ros_odometry">
-        <ros>
-          <namespace>${namespace}</namespace>
-        </ros>
-        <frame_name>world</frame_name>
-        <body_name>base_footprint</body_name>
-        <topic_name>ground_truth_odom</topic_name>
-        <update_rate>100.0</update_rate>
-      </plugin>
+      <xacro:if value="${gazebo_version == 'classic'}">
+        <plugin filename="libgazebo_world_odometry.so" name="gazebo_ros_odometry">
+          <ros>
+            <namespace>${namespace}</namespace>
+          </ros>
+          <frame_name>world</frame_name>
+          <body_name>base_footprint</body_name>
+          <topic_name>ground_truth_odom</topic_name>
+          <update_rate>100.0</update_rate>
+        </plugin>
+      </xacro:if>
     </gazebo>
   </xacro:macro>

File: pmb2_description/urdf/base/base_sensors.urdf.xacro (robot description, xacro)
@@ -63,11 +63,23 @@
     <!-- Sonars -->
     <xacro:if value="${has_sonars}">
-      <xacro:range_sensor name="${name}_sonar_03" parent="${name}_link" ros_topic="sonar_${name}" update_rate="5" maxRange="1.0" minRange="0.02" fov="0.5" radiation="ultrasound">
+      <!-- Gazebo: use numbered topics to visualize independently -->
+      <xacro:if value="${gazebo_version == 'gazebo'}">
+        <xacro:property name="sonar_topic_01" value="sonar_${name}_01"/>
+        <xacro:property name="sonar_topic_02" value="sonar_${name}_02"/>
+        <xacro:property name="sonar_topic_03" value="sonar_${name}_03"/>
+      </xacro:if>
+      <!-- Gazebo classic: all use same topic -->
+      <xacro:if value="${gazebo_version == 'classic'}">
+        <xacro:property name="sonar_topic_01" value="sonar_${name}"/>
+        <xacro:property name="sonar_topic_02" value="sonar_${name}"/>
+        <xacro:property name="sonar_topic_03" value="sonar_${name}"/>
+      </xacro:if>
+      <xacro:range_sensor name="${name}_sonar_03" parent="${name}_link" ros_topic="${sonar_topic_03}" update_rate="5" maxRange="1.0" minRange="0.02" fov="0.5" radiation="ultrasound">
         <origin xyz="-0.183 0.183 0.173" rpy="0 0 ${135 * deg_to_rad}"/>
       </xacro:range_sensor>
-      <xacro:range_sensor name="${name}_sonar_02" parent="${name}_link" ros_topic="sonar_${name}" update_rate="5" maxRange="1.0" minRange="0.02" fov="0.5" radiation="ultrasound">
+      <xacro:range_sensor name="${name}_sonar_02" parent="${name}_link" ros_topic="${sonar_topic_02}" update_rate="5" maxRange="1.0" minRange="0.02" fov="0.5" radiation="ultrasound">
         <origin xyz="-0.259 0.0 0.173" rpy="0 0 ${180 * deg_to_rad}"/>
       </xacro:range_sensor>
-      <xacro:range_sensor name="${name}_sonar_01" parent="${name}_link" ros_topic="sonar_${name}" update_rate="5" maxRange="1.0" minRange="0.02" fov="0.5" radiation="ultrasound">
+      <xacro:range_sensor name="${name}_sonar_01" parent="${name}_link" ros_topic="${sonar_topic_01}" update_rate="5" maxRange="1.0" minRange="0.02" fov="0.5" radiation="ultrasound">
         <origin xyz="-0.183 -0.183 0.173" rpy="0 0 ${225 * deg_to_rad}"/>
       </xacro:range_sensor>
